Commit message: Update UR5 LEAP models and validation scripts

File: source/ur5_leap/assets/combined/ur5_leap_right/urdf/ur5_leap_right.urdf (robot description, URDF)
Before this commit: robot ur5_cb3_leap_v1_right, 30 links, 29 joints
Links:
- removed link mounting_adapter
- added link ee_link
Joints:
- removed joint adapter_to_palm
- removed joint flange_to_adapter
- added joint ee_fixed_joint: type fixed, parent wrist_3_link, child ee_link, origin xyz=0.0 0.0823 0.0 rpy=0.0 0.0 1.57079632679
- added joint mount_joint: type fixed, parent ee_link, child palm_lower, origin xyz=0.0 0.03 0.06 rpy=3.14159 -1.57079 3.14159
